File: pcb_v2.3-unrouted.sch (EAGLE design)
At the start: 53 parts, among them J1 PJ301_THONKICONN6, J2 PJ301_THONKICONN6, J3 PJ301_THONKICONN6, J4 PJ301_THONKICONN6, U1 MCP6004, U2 TL074_SMD, U5 TL074

Commit message: route board
Connections:
- net NC renamed SV2_2
- new net N$16: U$1.VCC/+
- net 3V: no longer U$1.VCC/+
Changed lines of the file:
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@@
 <attribute name="SPICEPREFIX" value="G"/>
 </part>
+<part name="12V1" library="supply2" library_urn="urn:adsk.eagle:library:372" deviceset="V+" device=""/>
 <part name="GND22" library="SparkFun" deviceset="GND" device="">
 <attribute name="SPICEGROUND" value=""/>
@@
 <instance part="-12V" gate="1" x="60.96" y="116.84"/>
 <instance part="GND21" gate="1" x="99.06" y="119.38" rot="R180"/>
+<instance part="12V1" gate="1" x="71.12" y="119.38"/>
 <instance part="GND22" gate="1" x="88.9" y="184.15"/>
 <instance part="U$1" gate="G$1" x="130.81" y="158.75"/>
-<instance part="GND23" gate="1" x="115.57" y="138.43"/>
+<instance part="GND23" gate="1" x="118.11" y="138.43"/>
 <instance part="SW2" gate="S" x="214.63" y="151.13"/>
 <instance part="GND54" gate="1" x="207.01" y="143.51"/>
@@
 </segment>
 <segment>
+<pinref part="U$1" gate="G$1" pin="SHIELD@2"/>
+<wire x1="123.19" y1="146.05" x2="118.11" y2="146.05" width="0.1524" layer="91"/>
+<pinref part="GND23" gate="1" pin="GND"/>
+<wire x1="118.11" y1="146.05" x2="118.11" y2="140.97" width="0.1524" layer="91"/>
+<pinref part="U$1" gate="G$1" pin="SHIELD@1"/>
+<wire x1="123.19" y1="148.59" x2="118.11" y2="148.59" width="0.1524" layer="91"/>
+<wire x1="118.11" y1="148.59" x2="118.11" y2="140.97" width="0.1524" layer="91"/>
+<pinref part="U$1" gate="G$1" pin="GND"/>
+<wire x1="123.19" y1="158.75" x2="118.11" y2="158.75" width="0.1524" layer="91"/>
+<wire x1="118.11" y1="158.75" x2="118.11" y2="140.97" width="0.1524" layer="91"/>
+</segment>
+<segment>
 <wire x1="209.55" y1="151.13" x2="207.01" y2="151.13" width="0.1524" layer="91"/>
 <wire x1="207.01" y1="151.13" x2="207.01" y2="148.59" width="0.1524" layer="91"/>
@@
 <pinref part="GND22" gate="1" pin="GND"/>
 <wire x1="88.9" y1="190.5" x2="88.9" y2="186.69" width="0.1524" layer="91"/>
-</segment>
-<segment>
-<pinref part="U$1" gate="G$1" pin="SHIELD@2"/>
-<wire x1="123.19" y1="146.05" x2="115.57" y2="146.05" width="0.1524" layer="91"/>
-<pinref part="GND23" gate="1" pin="GND"/>
-<wire x1="115.57" y1="146.05" x2="115.57" y2="140.97" width="0.1524" layer="91"/>
-<pinref part="U$1" gate="G$1" pin="SHIELD@1"/>
-<wire x1="123.19" y1="148.59" x2="115.57" y2="148.59" width="0.1524" layer="91"/>
-<wire x1="115.57" y1="148.59" x2="115.57" y2="146.05" width="0.1524" layer="91"/>
-<junction x="115.57" y="146.05"/>
-<pinref part="U$1" gate="G$1" pin="GND"/>
-<wire x1="123.19" y1="158.75" x2="115.57" y2="158.75" width="0.1524" layer="91"/>
-<wire x1="115.57" y1="158.75" x2="115.57" y2="148.59" width="0.1524" layer="91"/>
-<junction x="115.57" y="148.59"/>
 </segment>
 </net>
@@
 </segment>
 <segment>
+<pinref part="12V1" gate="1" pin="V+"/>
 <wire x1="71.12" y1="116.84" x2="71.12" y2="106.68" width="0.1524" layer="91"/>
 <label x="71.12" y="111.76" size="1.778" layer="95" rot="R90"/>
@@
 <label x="118.11" y="163.83" size="1.524" layer="95" rot="R180" xref="yes"/>
 </segment>
-<segment>
-<pinref part="U$1" gate="G$1" pin="VCC/+"/>
-<wire x1="118.11" y1="163.83" x2="123.19" y2="163.83" width="0.1524" layer="91"/>
-</segment>
 </net>
 <net name="LOW_OUT" class="0">
 <segment>
-<wire x1="144.78" y1="25.4" x2="133.858" y2="25.4" width="0.1524" layer="91"/>
+<wire x1="140.208" y1="25.4" x2="133.858" y2="25.4" width="0.1524" layer="91"/>
 <pinref part="R5" gate="G$1" pin="2"/>
 <wire x1="121.92" y1="88.9" x2="133.858" y2="88.9" width="0.1524" layer="91"/>
 <wire x1="133.858" y1="88.9" x2="133.858" y2="25.4" width="0.1524" layer="91"/>
+<wire x1="144.78" y1="25.4" x2="140.208" y2="25.4" width="0.1524" layer="91"/>
 </segment>
 <segment>
@@
 <net name="HIGH_OUT" class="0">
 <segment>
-<wire x1="144.78" y1="15.24" x2="130.048" y2="15.24" width="0.1524" layer="91"/>
+<wire x1="140.208" y1="15.24" x2="130.048" y2="15.24" width="0.1524" layer="91"/>
 <pinref part="R17" gate="G$1" pin="2"/>
 <wire x1="121.92" y1="-2.54" x2="130.048" y2="-2.54" width="0.1524" layer="91"/>
 <wire x1="130.048" y1="-2.54" x2="130.048" y2="15.24" width="0.1524" layer="91"/>
+<wire x1="140.208" y1="15.24" x2="144.78" y2="15.24" width="0.1524" layer="91"/>
 </segment>
 <segment>
@@
 <segment>
 <pinref part="R23" gate="G$1" pin="2"/>
-<wire x1="121.92" y1="-50.8" x2="134.112" y2="-50.8" width="0.1524" layer="91"/>
+<wire x1="121.92" y1="-50.8" x2="124.46" y2="-50.8" width="0.1524" layer="91"/>
+<wire x1="124.46" y1="-50.8" x2="134.112" y2="-50.8" width="0.1524" layer="91"/>
 <wire x1="134.112" y1="-50.8" x2="134.112" y2="10.16" width="0.1524" layer="91"/>
 <wire x1="134.112" y1="10.16" x2="144.78" y2="10.16" width="0.1524" layer="91"/>
@@
 <wire x1="109.22" y1="156.21" x2="109.22" y2="153.67" width="0.1524" layer="91"/>
 <pinref part="SV2" gate="G$1" pin="1"/>
+</segment>
+</net>
+<net name="N$16" class="0">
+<segment>
+<pinref part="U$1" gate="G$1" pin="VCC/+"/>
+<wire x1="118.11" y1="163.83" x2="123.19" y2="163.83" width="0.1524" layer="91"/>
 </segment>
 </net>
@@
 </segment>
 </net>
-<net name="NC" class="0">
+<net name="SV2_2" class="0">
 <segment>
 <pinref part="SV2" gate="G$1" pin="2"/>
